Commit message: committ

File: robutler_description_T3/urdf/robutler.urdf.xacro (robot description, xacro)
@@ -160,4 +160,32 @@
     </inertial>
   </link>
+  <!-- Adding joint for new (possibly rotating) rgb camera -->
+    <joint name="object_camera_joint" type="fixed">
+    <parent link="camera_rgb_frame"/>
+    <child link="object_joint"/>
+    <origin xyz="0 0 0" rpy="0 0 0"/>
+  </joint>
+  <link name="object_joint">
+    <visual>
+      <origin xyz="-0.23 0 0.1" rpy="0 0 0"/>
+      <geometry>
+        <cylinder length="0.200" radius="0.0055"/>
+      </geometry>
+      <material name="white"/>
+    </visual>
+    <collision>
+      <origin xyz="0.015 0 -0.0065" rpy="0 0 0"/>
+      <geometry>
+        <cylinder length="0.1" radius="0.0055"/>
+      </geometry>
+    </collision>
+    <inertial>
+      <mass value="0.114" />
+      <origin xyz="0 0 0" />
+      <inertia ixx="0.001" ixy="0.0" ixz="0.0"
+               iyy="0.001" iyz="0.0"
+               izz="0.001" />
+    </inertial>
+  </link>
   <joint name="camera_joint" type="fixed">
     <origin xyz="0.073 -0.011 0.084" rpy="0 0 0"/>

Commit message: comitt

File: robutler_description_T3/urdf/robutler.urdf.xacro (robot description, xacro)
@@ -160,32 +160,4 @@
     </inertial>
   </link>
-  <!-- Adding joint for new (possibly rotating) rgb camera -->
-    <joint name="object_camera_joint" type="fixed">
-    <parent link="camera_rgb_frame"/>
-    <child link="object_joint"/>
-    <origin xyz="0 0 0" rpy="0 0 0"/>
-  </joint>
-  <link name="object_joint">
-    <visual>
-      <origin xyz="-0.23 0 0.1" rpy="0 0 0"/>
-      <geometry>
-        <cylinder length="0.200" radius="0.0055"/>
-      </geometry>
-      <material name="white"/>
-    </visual>
-    <collision>
-      <origin xyz="0.015 0 -0.0065" rpy="0 0 0"/>
-      <geometry>
-        <cylinder length="0.1" radius="0.0055"/>
-      </geometry>
-    </collision>
-    <inertial>
-      <mass value="0.114" />
-      <origin xyz="0 0 0" />
-      <inertia ixx="0.001" ixy="0.0" ixz="0.0"
-               iyy="0.001" iyz="0.0"
-               izz="0.001" />
-    </inertial>
-  </link>
   <joint name="camera_joint" type="fixed">
     <origin xyz="0.073 -0.011 0.084" rpy="0 0 0"/>

File: robutler_description_T3/urdf/turtlebot3_manipulation_robot.urdf.xacro (robot description, xacro)
@@ -2,5 +2,5 @@
 <robot name="turtlebot3_manipulation" xmlns:xacro="http://ros.org/wiki/xacro">
   <!-- Include TurtleBot3 Waffle URDF -->
-  <xacro:include filename="$(find robutler_description_T3)/urdf/turtlebot3_waffle_pi_for_open_manipulator.urdf.xacro"/>
+  <xacro:include filename="$(find robutler_description_T3)/urdf/robutler.urdf.xacro"/>
   <!-- Include OpenMANIPULATOR URDF -->
   <xacro:include filename="$(find robutler_description_T3)/urdf/open_manipulator_x.urdf.xacro"/>

Commit message: commit

File: robutler_description_T3/urdf/robutler.urdf.xacro (robot description, xacro)
@@ -173,15 +173,3 @@
     </collision>
   </link>
-  <joint name="camera_rgb_joint" type="fixed">
-    <origin xyz="0.003 0.011 0.009" rpy="0 0 0"/>
-    <parent link="camera_link"/>
-    <child link="camera_rgb_frame"/>
-  </joint>
-  <link name="camera_rgb_frame"/>
-  <joint name="camera_rgb_optical_joint" type="fixed">
-    <origin xyz="0 0 0" rpy="-1.57 0 -1.57"/>
-    <parent link="camera_rgb_frame"/>
-    <child link="camera_rgb_optical_frame"/>
-  </joint>
-  <link name="camera_rgb_optical_frame"/>
 </robot>

Commit message: commit

File: robutler_description_T3/urdf/robutler.urdf.xacro (robot description, xacro)
@@ -140,5 +140,5 @@
   <link name="base_scan">
     <visual>
-      <origin xyz="0 0 0.0" rpy="0 0 0"/>
+      <origin xyz="0.055 0.00 0" rpy="0 0 0"/>
       <geometry>
         <mesh filename="package://turtlebot3_description/meshes/sensors/lds.stl" scale="0.001 0.001 0.001"/>

Commit message: commit

File: robutler_description_T3/urdf/robutler.urdf.xacro (robot description, xacro)
@@ -167,5 +167,5 @@
   <link name="camera_link">
     <collision>
-      <origin xyz="0.005 0.011 0.013" rpy="0 0 0"/>
+      <origin xyz="0.005 0.011 0.013" rpy="-1.57 0 -1.57"/>
       <geometry>
         <box size="0.015 0.030 0.027"/>
@@ -173,3 +173,15 @@
     </collision>
   </link>
+  <joint name="camera_rgb_joint" type="fixed">
+    <origin xyz="0.003 0.011 0.009" rpy="0 0 0"/>
+    <parent link="camera_link"/>
+    <child link="camera_rgb_frame"/>
+  </joint>
+  <link name="camera_rgb_frame"/>
+  <joint name="camera_rgb_optical_joint" type="fixed">
+    <origin xyz="0 0 0" rpy="-1.57 0 -1.57"/>
+    <parent link="camera_link"/>
+    <child link="camera_rgb_optical_frame"/>
+  </joint>
+  <link name="camera_rgb_optical_frame"/>
 </robot>
