Commit message: commit

File: robutler_description_T3/urdf/open_manipulator_x.gazebo.xacro (robot description, xacro)
@@ -29,5 +29,5 @@
   <!-- end effector link -->
   <gazebo reference="end_effector_link">
-    <material>Gazebo/Red</material>
+    <material>Gazebo/Green</material>
   </gazebo>
   <!-- ros_control plugin -->

File: robutler_description_T3/urdf/open_manipulator_x.urdf.xacro (robot description, xacro)
@@ -232,5 +232,5 @@
         <box size="0.01 0.01 0.01" />
       </geometry>
-      <material name="red"/>
+      <material name="green"/>
      </visual>
     <inertial>
