Commit message: comitt

File: robutler_description_T3/urdf/open_manipulator_x.urdf.xacro (robot description, xacro)
@@ -156,4 +156,29 @@
     </inertial>
   </link>
+  <joint name="camera_joint_grip" type="fixed">
+    <origin xyz="0.073 -0.011 0.084" rpy="0 0 0"/>
+    <parent link="link5"/>
+    <child link="camera_link_grip"/>
+  </joint>
+  <link name="camera_link_grip">
+    <collision>
+      <origin xyz="0.005 0.011 0.013" rpy="-1.57 0 -1.57"/>
+      <geometry>
+        <box size="0.015 0.030 0.027"/>
+      </geometry>
+    </collision>
+  </link>
+  <joint name="camera_rgb_joint_grip" type="fixed">
+    <origin xyz="0.003 0.011 0.009" rpy="0 0 0"/>
+    <parent link="camera_link_grip"/>
+    <child link="camera_rgb_frame_grip"/>
+  </joint>
+  <link name="camera_rgb_frame_grip"/>
+  <joint name="camera_rgb_optical_joint_grip" type="fixed">
+    <origin xyz="0 0 0" rpy="-1.57 0 -1.57"/>
+    <parent link="camera_link_grip"/>
+    <child link="camera_rgb_optical_frame_grip"/>
+  </joint>
+  <link name="camera_rgb_optical_frame_grip"/>
   <!--  Gripper link -->
   <link name="gripper_link">

Commit message: camera for gripper added

File: robutler_description_T3/urdf/open_manipulator_x.urdf.xacro (robot description, xacro)
@@ -156,29 +156,4 @@
     </inertial>
   </link>
-  <joint name="camera_joint_grip" type="fixed">
-    <origin xyz="0.073 -0.011 0.084" rpy="0 0 0"/>
-    <parent link="link5"/>
-    <child link="camera_link_grip"/>
-  </joint>
-  <link name="camera_link_grip">
-    <collision>
-      <origin xyz="0.005 0.011 0.013" rpy="-1.57 0 -1.57"/>
-      <geometry>
-        <box size="0.015 0.030 0.027"/>
-      </geometry>
-    </collision>
-  </link>
-  <joint name="camera_rgb_joint_grip" type="fixed">
-    <origin xyz="0.003 0.011 0.009" rpy="0 0 0"/>
-    <parent link="camera_link_grip"/>
-    <child link="camera_rgb_frame_grip"/>
-  </joint>
-  <link name="camera_rgb_frame_grip"/>
-  <joint name="camera_rgb_optical_joint_grip" type="fixed">
-    <origin xyz="0 0 0" rpy="-1.57 0 -1.57"/>
-    <parent link="camera_link_grip"/>
-    <child link="camera_rgb_optical_frame_grip"/>
-  </joint>
-  <link name="camera_rgb_optical_frame_grip"/>
   <!--  Gripper link -->
   <link name="gripper_link">
@@ -267,3 +242,28 @@
     </inertial>
   </link>
+<joint name="camera_joint_grip" type="fixed">
+    <origin xyz="0 0.021 0.02" rpy="0 0 0"/>
+    <parent link="gripper_link_sub"/>
+    <child link="camera_link_grip"/>
+  </joint>
+  <link name="camera_link_grip">
+    <collision>
+      <origin xyz="0 0.021 0.013" rpy="-1.57 0 -1.57"/>
+      <geometry>
+        <box size="0.015 0.030 0.027"/>
+      </geometry>
+    </collision>
+  </link>
+  <joint name="camera_rgb_joint_grip" type="fixed">
+    <origin xyz="0 0 0.0013" rpy="0 0 0"/>
+    <parent link="camera_link_grip"/>
+    <child link="camera_rgb_frame_grip"/>
+  </joint>
+  <link name="camera_rgb_frame_grip"/>
+  <joint name="camera_rgb_optical_joint_grip" type="fixed">
+    <origin xyz="0 0 0" rpy="-1.57 0 -1.57"/>
+    <parent link="camera_link_grip"/>
+    <child link="camera_rgb_optical_frame_grip"/>
+  </joint>
+  <link name="camera_rgb_optical_frame_grip"/>
 </robot>

Commit message: commit

File: robutler_description_T3/urdf/open_manipulator_x.urdf.xacro (robot description, xacro)
@@ -12,5 +12,5 @@
         <mesh filename="package://robutler_description_T3/meshes/chain_link1.stl" scale="0.001 0.001 0.001"/>
       </geometry>
-      <material name="grey"/>
+      <material name="white"/>
     </visual>
     <collision>
@@ -43,5 +43,5 @@
         <mesh filename="package://robutler_description_T3/meshes/chain_link2.stl" scale="0.001 0.001 0.001"/>
       </geometry>
-      <material name="grey"/>
+      <material name="white"/>
     </visual>
     <collision>
@@ -74,5 +74,5 @@
         <mesh filename="package://robutler_description_T3/meshes/chain_link3.stl" scale="0.001 0.001 0.001"/>
       </geometry>
-      <material name="grey"/>
+      <material name="white"/>
     </visual>
     <collision>
@@ -105,5 +105,5 @@
         <mesh filename="package://robutler_description_T3/meshes/chain_link4.stl" scale="0.001 0.001 0.001"/>
       </geometry>
-      <material name="grey"/>
+      <material name="white"/>
     </visual>
     <collision>
@@ -136,5 +136,5 @@
         <mesh filename="package://robutler_description_T3/meshes/chain_link5.stl" scale="0.001 0.001 0.001"/>
       </geometry>
-      <material name="grey"/>
+      <material name="white"/>
     </visual>
     <collision>
@@ -163,5 +163,5 @@
         <mesh filename="package://robutler_description_T3/meshes/chain_link_grip_l.stl" scale="0.001 0.001 0.001"/>
       </geometry>
-      <material name="grey"/>
+      <material name="white"/>
     </visual>
     <collision>
@@ -194,5 +194,5 @@
         <mesh filename="package://robutler_description_T3/meshes/chain_link_grip_r.stl" scale="0.001 0.001 0.001"/>
       </geometry>
-      <material name="grey"/>
+      <material name="white"/>
     </visual>
     <collision>

File: robutler_description_T3/urdf/robutler.urdf.xacro (robot description, xacro)
@@ -15,5 +15,5 @@
         <mesh filename="package://turtlebot3_description/meshes/bases/waffle_pi_base.stl" scale="0.001 0.001 0.001"/>
       </geometry>
-      <material name="light_black"/>
+      <material name="red"/>
     </visual>
     <collision>
@@ -144,5 +144,5 @@
         <mesh filename="package://turtlebot3_description/meshes/sensors/lds.stl" scale="0.001 0.001 0.001"/>
       </geometry>
-      <material name="dark"/>
+      <material name="blue"/>
     </visual>
     <collision>
